File: board_design/daughter boards/3wireducer_daughter/3wireducer_daughter.sch (KiCad schematic (older format))
At the start: 9 parts, among them J1 Conn_01x09_Male, J2 Conn_01x03

Commit message: first MX export
Connections:
- net +5V: now reaches J1.2 (Pin_2), JP1.1
- net +12C: now reaches J1.4 (Pin_4), JP2.1
- net +28V: now reaches J1.5 (Pin_5), JP3.1
- net sig_out: now reaches C1.1, J1.9 (Pin_9), R1.2, R2.1
- net sig_in: now reaches J2.3 (Pin_3), R1.1
- net exc+: now reaches F1.1, J2.1 (Pin_1)
Other:
- moved on the sheet: C1, J1, J2, R1, R2
