File: board_design/daughter boards/thermocouple_daughter/thermocouple_daughter.kicad_pcb (KiCad board)
At the start: 2 copper layers, 20.3 x 38.6 mm, 11 parts, among them J1 Conn_01x09_Male, J2 Conn_01x02, U1 AD8613, U2 AD8495

Commit message: push for jack
Changed lines of the file:
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@@
     (add_net sig)
+  )
+  (module davenport_kicad_footprints:PCC-OST (layer F.Cu)
+    (at 157.734 73.533)
+    (fp_text reference J2 (at -0.127 6.858) (layer F.SilkS)
+      (effects (font (size 1 1) (thickness 0.15)))
+    )
+    (fp_text value Conn_01x02 (at 0 -7.612) (layer F.Fab)
+      (effects (font (size 1 1) (thickness 0.15)))
+    )
+    (fp_line (start 0.508 -1.016) (end 0 -2.032) (layer F.CrtYd) (width 0.12))
+    (fp_line (start -0.508 -1.016) (end 0.508 -1.016) (layer F.CrtYd) (width 0.12))
+    (fp_line (start 0 -2.032) (end -0.508 -1.016) (layer F.CrtYd) (width 0.12))
+    (fp_line (start -10.16 -2.032) (end -10.16 -1.524) (layer F.CrtYd) (width 0.12))
+    (fp_line (start 10.16 -2.032) (end -10.16 -2.032) (layer F.CrtYd) (width 0.12))
+    (fp_line (start 10.16 15.24) (end 10.16 -2.032) (layer F.CrtYd) (width 0.12))
+    (fp_line (start -10.16 15.24) (end 10.16 15.24) (layer F.CrtYd) (width 0.12))
+    (fp_line (start -10.16 -1.524) (end -10.16 15.24) (layer F.CrtYd) (width 0.12))
+    (pad 2 thru_hole circle (at 6.8 13.5) (size 3 3) (drill 1.77) (layers *.Cu *.Mask)
+      (net 1 "Net-(C1-Pad1)"))
+    (pad 1 thru_hole circle (at -6.8 13.5) (size 3 3) (drill 1.77) (layers *.Cu *.Mask)
+      (net 2 "Net-(C1-Pad2)"))
+    (pad "" thru_hole circle (at 7.9 0) (size 2.5 2.5) (drill 1.77) (layers *.Cu *.Mask))
+    (pad "" thru_hole circle (at -7.9 0) (size 2.5 2.5) (drill 1.77) (layers *.Cu *.Mask))
   )
   (module davenport_kicad_footprints:logo-bss (layer B.Cu)
@@
     )
   )
-  (module davenport_kicad_footprints:PCC-OST (layer F.Cu)
-    (at 157.734 73.533)
-    (fp_text reference J2 (at -0.127 6.858) (layer F.SilkS)
-      (effects (font (size 1 1) (thickness 0.15)))
-    )
-    (fp_text value Conn_01x02 (at 0 -7.612) (layer F.Fab)
-      (effects (font (size 1 1) (thickness 0.15)))
-    )
-    (fp_line (start -10.16 -1.524) (end -10.16 15.24) (layer F.CrtYd) (width 0.12))
-    (fp_line (start -10.16 15.24) (end 10.16 15.24) (layer F.CrtYd) (width 0.12))
-    (fp_line (start 10.16 15.24) (end 10.16 -2.032) (layer F.CrtYd) (width 0.12))
-    (fp_line (start 10.16 -2.032) (end -10.16 -2.032) (layer F.CrtYd) (width 0.12))
-    (fp_line (start -10.16 -2.032) (end -10.16 -1.524) (layer F.CrtYd) (width 0.12))
-    (fp_line (start 0 -2.032) (end -0.508 -1.016) (layer F.CrtYd) (width 0.12))
-    (fp_line (start -0.508 -1.016) (end 0.508 -1.016) (layer F.CrtYd) (width 0.12))
-    (fp_line (start 0.508 -1.016) (end 0 -2.032) (layer F.CrtYd) (width 0.12))
-    (pad "" thru_hole circle (at -7.9 0) (size 1.77 1.77) (drill 0.762) (layers *.Cu *.Mask))
-    (pad "" thru_hole circle (at 7.9 0) (size 1.77 1.77) (drill 0.762) (layers *.Cu *.Mask))
-    (pad 1 thru_hole circle (at -6.8 13.5) (size 1.77 1.77) (drill 0.762) (layers *.Cu *.Mask)
-      (net 2 "Net-(C1-Pad2)"))
-    (pad 2 thru_hole circle (at 6.8 13.5) (size 1.77 1.77) (drill 0.762) (layers *.Cu *.Mask)
-      (net 1 "Net-(C1-Pad1)"))
-  )
   (module Resistor_SMD:R_0805_2012Metric (layer F.Cu)
