File: board_design/prop_support/power.sch (KiCad schematic (older format))
At the start: 48 parts, among them J2 GS2, J3 XT-60_female, U2 INA181, U3 LM1117-3.3, U4 LT1930, U5 LM1117-5.0

Commit message: first MX export
Other:
- note added: "Bus Telemetry"
- moved on the sheet: C12, C13, C14, C15, C16, C17, D1, D2, D3, D4, FB1, J3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
