File: board_design/prop_support/valve_channel_nosense.sch (KiCad schematic (older format))
At the start: 10 parts, among them Q1 MMBT3904, Q2 Q_PMOS_GDS

Commit message: first MX export
Changed lines of the file:
@@
 $Descr A4 11693 8268
 encoding utf-8
-Sheet 6 14
+Sheet 5 14
 Title "Prop Support Board"
 Date "2019-03-27"
@@
 AR Path="/5C9C50FB/5CA19CF4/596707F4" Ref="#PWR0196"  Part="1"
 AR Path="/5C9C50FB/5CA19CFA/596707F4" Ref="#PWR0204"  Part="1"
-F 0 "#PWR0156" H 6800 3050 50  0001 C CNN
+F 0 "#PWR0148" H 6800 3050 50  0001 C CNN
 F 1 "+12V" H 6800 3340 50  0000 C CNN
 F 2 "" H 6800 3200 50  0001 C CNN
@@
 AR Path="/5C9C50FB/5CA19CF4/59671CF5" Ref="#PWR0197"  Part="1"
 AR Path="/5C9C50FB/5CA19CFA/59671CF5" Ref="#PWR0205"  Part="1"
-F 0 "#PWR0157" H 5600 3675 50  0001 C CNN
+F 0 "#PWR0149" H 5600 3675 50  0001 C CNN
 F 1 "GND" H 5600 3775 50  0000 C CNN
 F 2 "" H 5600 3925 50  0001 C CNN
@@
 AR Path="/5C9C50FB/5CA19CF4/59672FA2" Ref="R50"  Part="1"
 AR Path="/5C9C50FB/5CA19CFA/59672FA2" Ref="R55"  Part="1"
-F 0 "R25" V 4655 3950 50  0000 C CNN
+F 0 "R20" V 4655 3950 50  0000 C CNN
 F 1 "1k" V 4575 3950 50  0000 C CNN
 F 2 "Resistor_SMD:R_0805_2012Metric" V 4505 3950 50  0001 C CNN
@@
 AR Path="/5C9C50FB/5CA19CF4/59673012" Ref="R51"  Part="1"
 AR Path="/5C9C50FB/5CA19CFA/59673012" Ref="R56"  Part="1"
-F 0 "R26" V 4955 3650 50  0000 C CNN
+F 0 "R21" V 4955 3650 50  0000 C CNN
 F 1 "1k" V 4875 3650 50  0000 C CNN
 F 2 "Resistor_SMD:R_0805_2012Metric" V 4805 3650 50  0001 C CNN
@@
 AR Path="/5C9C50FB/5CA19CF4/59673D60" Ref="R53"  Part="1"
 AR Path="/5C9C50FB/5CA19CFA/59673D60" Ref="R58"  Part="1"
-F 0 "R28" V 5680 3225 50  0000 C CNN
+F 0 "R23" V 5680 3225 50  0000 C CNN
 F 1 "1k" V 5600 3225 50  0000 C CNN
 F 2 "Resistor_SMD:R_0805_2012Metric" V 5530 3225 50  0001 C CNN
@@
 AR Path="/5C9C50FB/5CA19CF4/59673EA8" Ref="#PWR0198"  Part="1"
 AR Path="/5C9C50FB/5CA19CFA/59673EA8" Ref="#PWR0206"  Part="1"
-F 0 "#PWR0158" H 4575 3900 50  0001 C CNN
+F 0 "#PWR0150" H 4575 3900 50  0001 C CNN
 F 1 "GND" H 4575 4000 50  0000 C CNN
 F 2 "" H 4575 4150 50  0001 C CNN
@@
 AR Path="/5C9C50FB/5CA19CF4/59674072" Ref="#PWR0199"  Part="1"
 AR Path="/5C9C50FB/5CA19CFA/59674072" Ref="#PWR0207"  Part="1"
-F 0 "#PWR0159" H 5600 2875 50  0001 C CNN
+F 0 "#PWR0151" H 5600 2875 50  0001 C CNN
 F 1 "+12V" H 5600 3165 50  0000 C CNN
 F 2 "" H 5600 3025 50  0001 C CNN
@@
 AR Path="/5C9C50FB/5CA19CF4/5A1E0B4E" Ref="Q14"  Part="1"
 AR Path="/5C9C50FB/5CA19CFA/5A1E0B4E" Ref="Q16"  Part="1"
-F 0 "Q4" H 6900 3450 50  0000 L CNN
+F 0 "Q2" H 6900 3450 50  0000 L CNN
 F 1 "Q_PMOS_GDS" H 6900 3350 50  0000 L CNN
 F 2 "Package_TO_SOT_SMD:TO-252-2" H 6900 3500 50  0001 C CNN
@@
 AR Path="/5C9C50FB/5CA19CF4/5C9E97B4" Ref="#PWR0215"  Part="1"
 AR Path="/5C9C50FB/5CA19CFA/5C9E97B4" Ref="#PWR0216"  Part="1"
-F 0 "#PWR0209" H 6325 4575 50  0001 C CNN
+F 0 "#PWR0208" H 6325 4575 50  0001 C CNN
 F 1 "GNDPWR" H 6329 4621 50  0000 C CNN
 F 2 "" H 6325 4725 50  0001 C CNN
@@
 AR Path="/5C9C50FB/5CA19CF4/5CA173EE" Ref="#PWR0203"  Part="1"
 AR Path="/5C9C50FB/5CA19CFA/5CA173EE" Ref="#PWR0211"  Part="1"
-F 0 "#PWR0163" H 5100 2275 50  0001 C CNN
+F 0 "#PWR0155" H 5100 2275 50  0001 C CNN
 F 1 "+3.3V" H 5115 2598 50  0000 C CNN
 F 2 "" H 5100 2425 50  0001 C CNN
@@
 AR Path="/5C9C50FB/5CA19CF4/5CA14C75" Ref="S7"  Part="1"
 AR Path="/5C9C50FB/5CA19CFA/5CA14C75" Ref="S8"  Part="1"
-F 0 "S2" V 5253 2537 60  0000 R CNN
+F 0 "S1" V 5253 2537 60  0000 R CNN
 F 1 "100SP3T1B1M2QE" V 5375 2525 60  0000 R CNN
 F 2 "digikey-footprints:Toggle_Switch_100SP1T1B4M2QE" H -2700 3475 60  0001 L CNN
@@
 AR Path="/5C9C50FB/5CA19CF4/5CA10627" Ref="R52"  Part="1"
 AR Path="/5C9C50FB/5CA19CFA/5CA10627" Ref="R57"  Part="1"
-F 0 "R27" V 5280 3175 50  0000 C CNN
+F 0 "R22" V 5280 3175 50  0000 C CNN
 F 1 "1k" V 5200 3175 50  0000 C CNN
 F 2 "Resistor_SMD:R_0805_2012Metric" V 5130 3175 50  0001 C CNN
@@
 AR Path="/5C9C50FB/5CA19CF4/59673A80" Ref="Q13"  Part="1"
 AR Path="/5C9C50FB/5CA19CFA/59673A80" Ref="Q15"  Part="1"
-F 0 "Q3" H 5700 3725 50  0000 L CNN
+F 0 "Q1" H 5700 3725 50  0000 L CNN
 F 1 "MMBT3904" H 5100 3450 50  0000 L CNN
 F 2 "Package_TO_SOT_SMD:SOT-23" H 5700 3575 50  0001 L CIN
@@
 AR Path="/5C9C50FB/5CA19CF4/5C9FCEF3" Ref="R54"  Part="1"
 AR Path="/5C9C50FB/5CA19CFA/5C9FCEF3" Ref="R59"  Part="1"
-F 0 "R29" V 6225 4125 50  0000 C CNN
+F 0 "R24" V 6225 4125 50  0000 C CNN
 F 1 "1k" V 6325 4100 50  0000 C CNN
 F 2 "Resistor_SMD:R_0805_2012Metric" V 6255 4100 50  0001 C CNN
@@
 AR Path="/5C9C50FB/5CA19CF4/5C9D8F25" Ref="D18"  Part="1"
 AR Path="/5C9C50FB/5CA19CFA/5C9D8F25" Ref="D20"  Part="1"
-F 0 "D8" V 6364 4408 50  0000 R CNN
+F 0 "D6" V 6364 4408 50  0000 R CNN
 F 1 "LED" V 6273 4408 50  0000 R CNN
 F 2 "LED_SMD:LED_0805_2012Metric" H 6325 4525 50  0001 C CNN
@@
 AR Path="/5C9C50FB/5CA19CF4/59730D47" Ref="D19"  Part="1"
 AR Path="/5C9C50FB/5CA19CFA/59730D47" Ref="D21"  Part="1"
-F 0 "D9" H 6800 4550 50  0000 C CNN
+F 0 "D7" H 6800 4550 50  0000 C CNN
 F 1 "D" H 6800 4350 50  0000 C CNN
 F 2 "davenport_kicad_footprints:SODFL4725X110N" H 6800 4450 50  0001 C CNN
