File: board_design/prop_support/prop_support.kicad_pcb (KiCad board)
At the start: 2 copper layers, 219.7 x 106.7 mm, 191 parts, among them J1 Conn_02x03_Counter_Clockwise, J10 Screw_Terminal_01x02, J11 Screw_Terminal_01x02, J12 Screw_Terminal_01x02, J13 Conn_01x09_Female, J14 Conn_01x09_Female, J15 Conn_01x09_Female, J16 Conn_01x09_Female, J17 Conn_01x09_Female, J18 Conn_01x09_Female, J19 Conn_01x09_Female, J2 GS2, J20 Conn_01x09_Female, J3 XT-60_female, J4 USB_B, J5 Screw_Terminal_01x02, J6 Screw_Terminal_01x02, J7 Screw_Terminal_01x02, J8 Screw_Terminal_01x02, J9 Screw_Terminal_01x02, Q1 MMBT3904, Q10 Q_PMOS_GDS, Q11 MMBT3904, Q12 Q_PMOS_GDS, Q13 MMBT3904, Q14 Q_PMOS_GDS, Q15 MMBT3904, Q16 Q_PMOS_GDS, Q2 Q_PMOS_GDS, Q3 MMBT3904, Q4 Q_PMOS_GDS, Q5 MMBT3904, Q6 Q_PMOS_GDS, Q7 MMBT3904, Q8 Q_PMOS_GDS, Q9 MMBT3904, SW1 SW_Push, U1 STM32F446RETx, U2 INA181, U3 LM1117-3.3, U4 LT1930, U5 LM1117-5.0, U6 FT232H, Y1 CX3225CA

Commit message: push for jack
Parts:
- added G***: LOGO, davenport_kicad_footprints:parrot, B.Cu at (119.8, 86.9)
- moved G*** 20.8 mm to (261.1, 130.8)
- moved R11 20.8 mm to (261.3, 82.0)
- moved R12 20.8 mm to (261.3, 78.2)
- moved R13 20.8 mm to (261.3, 74.4)
- moved R14 20.8 mm to (261.3, 70.6)
- moved Q12 20.8 mm to (129.0, 131.3)
- moved R40 20.8 mm to (146.1, 117.7)
- moved R49 20.8 mm to (131.9, 142.7)
- moved D20 20.8 mm to (82.1, 142.7)
- moved Q16 20.8 mm to (83.1, 131.8)
- moved C1 20.8 mm to (158.6, 92.3)
- moved C10 20.8 mm to (175.9, 97.0)
- moved C11 20.8 mm to (171.3, 79.0)
- moved C13 20.8 mm to (68.1, 100.8)
- moved C14 20.8 mm to (71.9, 94.5)
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